File: MotorDriverRev5.sch (KiCad schematic (older format))
At the start: 114 parts, among them J10 n/a, J15 Board_hole, J16 Board_hole, J17 Board_hole, J18 Board_hole, J19 Board_hole, J20 Board_hole, J3 Intel_LGA115x_holes, J5 CONN_01X06, J6 N/A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

Commit message: Updated libraries for using git
Parts:
- removed U?: DSPIC33EPXXXMC204/504, Housings_QFP:TQFP-44_10x10mm_Pitch0.8mm, symbol DSPIC33EPXXXMC204/504
- added U?: DSPIC33EPXXXMC204/504, Housings_QFP:TQFP-44_10x10mm_Pitch0.8mm, symbol DSPIC33EPXXXMC204/504
Changed lines of the file:
@@
 LIBS:contrib
 LIBS:valves
-LIBS:diode
+LIBS:Kicad_components_LJD
 LIBS:MotorDriverRev5-cache
 EELAYER 25 0
@@
 $Comp
 L DSPIC33EPXXXMC204/504 U?
-U 1 1 56E16B26
-P 5900 3500
-F 0 "U?" H 4350 4850 60  0000 C CNN
-F 1 "DSPIC33EPXXXMC204/504" H 4850 4750 60  0000 C CNN
-F 2 "Housings_QFP:TQFP-44_10x10mm_Pitch0.8mm" H 6400 4700 60  0000 C CNN
-F 3 "http://ww1.microchip.com/downloads/en/DeviceDoc/70000657H.pdf" H 6400 4700 60  0000 C CNN
-F 4 "DSPIC33EP128MC204-I/PT" H 5900 3500 60  0001 C CNN "manf#"
-	1    5900 3500
+U 1 1 56E62902
+P 5950 3200
+F 0 "U?" H 4400 4550 60  0000 C CNN
+F 1 "DSPIC33EPXXXMC204/504" H 4900 4450 60  0000 C CNN
+F 2 "Housings_QFP:TQFP-44_10x10mm_Pitch0.8mm" H 6100 5650 60  0001 C CNN
+F 3 "http://ww1.microchip.com/downloads/en/DeviceDoc/70000657H.pdf" H 6600 5500 60  0001 C CNN
+	1    5950 3200
 	1    0    0    -1
 $EndComp
